Commit message: update urdf

File: test/arm_v4.urdf (robot description, URDF)
Before this commit: robot arm_v2, 9 links, 8 joints
Links:
- link arm_link: geometry collision cylinder length=0.263 radius=0.0275; visual mesh filename=package://arm_v4/meshes/arm_link.STL
- link base_link: geometry collision cylinder length=0.07 radius=0.0325; visual mesh filename=package://arm_v4/meshes/base_link.STL
- link elbow_link: geometry collision cylinder length=0.05 radius=0.0325; visual mesh filename=package://arm_v4/meshes/elbow_link.STL
- link forearm_link: geometry collision cylinder length=0.142 radius=0.0275; visual mesh filename=package://arm_v4/meshes/forearm_link.STL
- link hand_link: geometry collision cylinder length=0.053 radius=0.0325; visual mesh filename=package://arm_v4/meshes/hand_link.STL
- link shoulder_link: geometry collision cylinder length=0.1675 radius=0.0325; visual mesh filename=package://arm_v4/meshes/shoulder_link.STL
- link wrist_link: geometry collision cylinder length=0.074 radius=0.0325; visual mesh filename=package://arm_v4/meshes/wrist_link.STL
